File: sensor/hardware/KiCAD/active_sender.kicad_pcb (KiCad board)
At the start: 2 copper layers, 83 x 80 mm, 27 parts, among them J1 220V0, J2 Buzzer, J3 Water Sensor, Q1 AO3400A, SW1 SW_Push, U1 ESP32-C3_SUPERMINI_TH, U2 Ai-Thinker-Ra-02, U3 HLK-PM12

Commit message: dev
Parts:
- added R10: 0R, Resistor_SMD:R_2512_6332Metric_Pad1.40x3.35mm_HandSolder, B.Cu at (97.0, 107.0)
- added SW2: SW_SPDT, custom_footprints:SS12D00, F.Cu at (92.0, 104.5)
- J3: footprint Connector_JST:JST_XH_B4B-XH-AM_1x04_P2.50mm_Vertical -> Connector_JST:JST_XH_S4B-XH-A-1_1x04_P2.50mm_Horizontal
- moved Q1 6.36 mm to (101.0, 100.0)
- moved J3 4.00 mm to (91.0, 114.0)
- moved REF** 3.00 mm to (68.0, 123.0)
- moved REF** 3.00 mm to (141.0, 123.0)
- moved D1 1.00 mm to (94.0, 97.0)
Connections:
- J3 pad 4: GNDPWR -> /MODE
Routing:
- net Net-(Q1-G): track 23.4 -> 16.2 mm
- net Net-(SW2-B): track 0.00 -> 5.25 mm
- net /MODE: track 0.00 -> 4.62 mm
- net Net-(U2-DIO0): track 11.0 -> 10.5 mm
- net /LORA_SCK: track 21.1 -> 21.6 mm
- net /LORA_RESET: track 71.9 -> 72.4 mm
- net /LORA_MOSI: track 26.6 -> 27.1 mm
- net /LORA_MISO: track 31.0 -> 31.5 mm
