File: sensor/hardware/KiCAD/active_sender.kicad_sch (KiCad schematic)
At the start: 22 parts, among them J1 220V0, J2 Buzzer, J3 Water Sensor, Q1 AO3400A, SW1 SW_Push, U1 ESP32-C3_SUPERMINI_TH, U2 Ai-Thinker-Ra-02, U3 HLK-PM12

Commit message: dev
Parts:
- added SW2: SW_SPDT, custom_footprints:SS12D00, symbol Switch:SW_SPDT
- J3: footprint Connector_JST:JST_XH_B4B-XH-AM_1x04_P2.50mm_Vertical -> Connector_JST:JST_XH_S4B-XH-A-1_1x04_P2.50mm_Horizontal
Connections:
- net 12V0: now also SW2.3 (C)
- net GNDPWR: now also SW2.1 (A); no longer J3.4 (Pin_4)
- new net MODE: J3.4 (Pin_4), SW2.2 (B)
Other:
- moved on the sheet: J3
