File: sensor/hardware/KiCAD/active_sender.kicad_sch (KiCad schematic)
At the start: 23 parts, among them J1 220V0, J2 Buzzer, J3 Water Sensor, Q1 AO3400A, SW1 SW_Push, SW2 SW_SPDT, U1 ESP32-C3_SUPERMINI_TH, U2 Ai-Thinker-Ra-02, U3 HLK-PM12

Commit message: dev
Parts:
- added F1: Fuse, Fuse:Fuseholder_Cylinder-5x20mm_Schurter_0031_8201_Horizontal_Open, symbol Device:Fuse
- added R10: 0R, Resistor_SMD:R_2512_6332Metric_Pad1.40x3.35mm_HandSolder, symbol Device:R
Connections:
- net 220V0: now also F1.2; no longer J1.1 (Pin_1)
- net MODE: now also R10.2; no longer SW2.2 (B)
- new net: R10.1, SW2.2 (B)
- new net: F1.1, J1.1 (Pin_1)
Other:
- moved on the sheet: J1
Changed lines of the file:
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@@
 	(wire
 		(pts
-			(xy 45.72 40.64) (xy 55.88 40.64)
+			(xy 33.02 40.64) (xy 55.88 40.64)
 		)
 		(stroke
@@
 	(wire
 		(pts
-			(xy 45.72 38.1) (xy 55.88 38.1)
+			(xy 33.02 38.1) (xy 36.83 38.1)
 		)
 		(stroke
@@
 	(wire
 		(pts
-			(xy 36.83 99.06) (xy 55.88 99.06)
+			(xy 36.83 99.06) (xy 45.72 99.06)
 		)
 		(stroke
@@
 	(wire
 		(pts
+			(xy 53.34 99.06) (xy 55.88 99.06)
+		)
+		(stroke
+			(width 0)
+			(type default)
+		)
+	)
+	(wire
+		(pts
 			(xy 52.07 66.04) (xy 52.07 69.85)
 		)
@@
 	(wire
 		(pts
+			(xy 44.45 38.1) (xy 55.88 38.1)
+		)
+		(stroke
+			(width 0)
+			(type default)
+		)
+	)
+	(wire
+		(pts
 			(xy 81.28 85.09) (xy 95.25 85.09)
 		)
@@
 	(symbol
 		(lib_id "Device:R")
+		(at 49.53 99.06 270)
+		(mirror x)
+		(unit 1)
+		(body_style 1)
+		(exclude_from_sim no)
+		(in_bom yes)
+		(on_board yes)
+		(in_pos_files yes)
+		(dnp no)
+		(property "Reference" "R10"
+			(at 49.53 103.378 90)
+			(show_name no)
+			(do_not_autoplace no)
+			(effects
+				(font
+					(size 1.27 1.27)
+				)
+			)
+		)
+		(property "Value" "0R"
+			(at 49.53 101.346 90)
+			(show_name no)
+			(do_not_autoplace no)
+			(effects
+				(font
+					(size 1.27 1.27)
+				)
+			)
+		)
+		(property "Footprint" "Resistor_SMD:R_2512_6332Metric_Pad1.40x3.35mm_HandSolder"
+			(at 49.53 100.838 90)
+			(hide yes)
+			(show_name no)
+			(do_not_autoplace no)
+			(effects
+				(font
+					(size 1.27 1.27)
+				)
+			)
+		)
+		(property "Datasheet" ""
+			(at 49.53 99.06 0)
+			(hide yes)
+			(show_name no)
+			(do_not_autoplace no)
+			(effects
+				(font
+					(size 1.27 1.27)
+				)
+			)
+		)
+		(property "Description" "Resistor"
+			(at 49.53 99.06 0)
+			(hide yes)
+			(show_name no)
+			(do_not_autoplace no)
+			(effects
+				(font
+					(size 1.27 1.27)
+				)
+			)
+		)
+		(pin "1"
+		)
+		(pin "2"
+		)
+		(instances
+			(project "active_sender"
+				(path "/0a63acd0-8ffb-408e-b0ed-0179bed06f72"
+					(reference "R10")
+					(unit 1)
+				)
+			)
+		)
+	)
+	(symbol
+		(lib_id "Device:R")
 		(at 157.48 81.28 0)
 		(mirror y)
@@
 	)
 	(symbol
-		(lib_id "Diode:SS34")
-		(at 57.15 64.77 270)
+		(lib_id "Device:Fuse")
+		(at 40.64 38.1 90)
 		(unit 1)
 		(body_style 1)
@@
 		(dnp no)
 		(fields_autoplaced yes)
-		(property "Reference" "D1"
-			(at 59.69 63.1824 90)
+		(property "Reference" "F1"
+			(at 40.64 31.75 90)
 			(show_name no)
 			(do_not_autoplace no)
@@
 					(size 1.27 1.27)
 				)
-				(justify left)
 			)
 		)
-		(property "Value" "SS34"
-			(at 59.69 65.7224 90)
+		(property "Value" "Fuse"
+			(at 40.64 34.29 90)
 			(show_name no)
 			(do_not_autoplace no)
@@
 					(size 1.27 1.27)
 				)
-				(justify left)
 			)
 		)
-		(property "Footprint" "Diode_SMD:D_SMA"
-			(at 52.705 64.77 0)
+		(property "Footprint" "Fuse:Fuseholder_Cylinder-5x20mm_Schurter_0031_8201_Horizontal_Open"
+			(at 40.64 39.878 90)
 			(hide yes)
 			(show_name no)
@@
 			)
 		)
-		(property "Datasheet" "https://www.vishay.com/docs/88751/ss32.pdf"
-			(at 57.15 64.77 0)
+		(property "Datasheet" ""
+			(at 40.64 38.1 0)
 			(hide yes)
 			(show_name no)
@@
 			)
 		)
-		(property "Description" "40V 3A Schottky Diode, SMA"
-			(at 57.15 64.77 0)
+		(property "Description" "Fuse"
+			(at 40.64 38.1 0)
 			(hide yes)
 			(show_name no)
@@
 			)
 		)
-		(pin "2"
-		)
 		(pin "1"
 		)
+		(pin "2"
+		)
 		(instances
 			(project "active_sender"
 				(path "/0a63acd0-8ffb-408e-b0ed-0179bed06f72"
-					(reference "D1")
+					(reference "F1")
 					(unit 1)
 				)
@@
 	)
 	(symbol
-		(lib_id "Switch:SW_SPDT")
-		(at 55.88 115.57 270)
+		(lib_id "Diode:SS34")
+		(at 57.15 64.77 270)
 		(unit 1)
 		(body_style 1)
@@
 		(dnp no)
 		(fields_autoplaced yes)
-		(property "Reference" "SW2"
-			(at 60.96 114.2999 90)
+		(property "Reference" "D1"
+			(at 59.69 63.1824 90)
 			(show_name no)
 			(do_not_autoplace no)
@@
 			)
 		)
-		(property "Value" "SW_SPDT"
-			(at 60.96 116.8399 90)
+		(property "Value" "SS34"
+			(at 59.69 65.7224 90)
 			(show_name no)
 			(do_not_autoplace no)
@@
 			)
 		)
-		(property "Footprint" "custom_footprints:SS12D00"
-			(at 55.88 115.57 0)
+		(property "Footprint" "Diode_SMD:D_SMA"
+			(at 52.705 64.77 0)
 			(hide yes)
 			(show_name no)
@@
 			)
 		)
-		(property "Datasheet" ""
-			(at 48.26 115.57 0)
+		(property "Datasheet" "https://www.vishay.com/docs/88751/ss32.pdf"
+			(at 57.15 64.77 0)
 			(hide yes)
 			(show_name no)
@@
 			)
 		)
-		(property "Description" "Switch, single pole double throw"
-			(at 55.88 115.57 0)
+		(property "Description" "40V 3A Schottky Diode, SMA"
+			(at 57.15 64.77 0)
 			(hide yes)
 			(show_name no)
@@
 			)
 		)
-		(pin "1"
-		)
-		(pin "3"
-		)
 		(pin "2"
 		)
+		(pin "1"
+		)
 		(instances
 			(project "active_sender"
 				(path "/0a63acd0-8ffb-408e-b0ed-0179bed06f72"
-					(reference "SW2")
+					(reference "D1")
 					(unit 1)
 				)
@@
 	)
 	(symbol
-		(lib_id "power:GNDPWR")
-		(at 33.02 80.01 0)
+		(lib_id "Switch:SW_SPDT")
+		(at 55.88 115.57 270)
 		(unit 1)
 		(body_style 1)
@@
 		(dnp no)
 		(fields_autoplaced yes)
-		(property "Reference" "#PWR015"
-			(at 33.02 85.09 0)
-			(hide yes)
+		(property "Reference" "SW2"
+			(at 60.96 114.2999 90)
 			(show_name no)
 			(do_not_autoplace no)
@@
 					(size 1.27 1.27)
 				)
+				(justify left)
 			)
 		)
-		(property "Value" "GNDPWR"
-			(at 32.893 83.82 0)
+		(property "Value" "SW_SPDT"
+			(at 60.96 116.8399 90)
 			(show_name no)
 			(do_not_autoplace no)
@@
 					(size 1.27 1.27)
 				)
+				(justify left)
 			)
 		)
-		(property "Footprint" ""
-			(at 33.02 81.28 0)
+		(property "Footprint" "custom_footprints:SS12D00"
+			(at 55.88 115.57 0)
 			(hide yes)
 			(show_name no)
@@
 		)
 		(property "Datasheet" ""
-			(at 33.02 81.28 0)
+			(at 48.26 115.57 0)
 			(hide yes)
 			(show_name no)
@@
 			)
 		)
-		(property "Description" "Power symbol creates a global label with name \"GNDPWR\" , global ground"
-			(at 33.02 80.01 0)
+		(property "Description" "Switch, single pole double throw"
+			(at 55.88 115.57 0)
 			(hide yes)
 			(show_name no)
@@
 		(pin "1"
 		)
+		(pin "3"
+		)
+		(pin "2"
+		)
 		(instances
 			(project "active_sender"
 				(path "/0a63acd0-8ffb-408e-b0ed-0179bed06f72"
-					(reference "#PWR015")
+					(reference "SW2")
 					(unit 1)
 				)
@@
 	(symbol
 		(lib_id "Connector:Screw_Terminal_01x02")
-		(at 40.64 38.1 0)
+		(at 27.94 38.1 0)
 		(mirror y)
 		(unit 1)
@@
 		(fields_autoplaced yes)
 		(property "Reference" "J1"
-			(at 40.64 31.75 0)
+			(at 27.94 31.75 0)
 			(show_name no)
 			(do_not_autoplace no)
@@
 		)
 		(property "Value" "220V0"
-			(at 40.64 34.29 0)
+			(at 27.94 34.29 0)
 			(show_name no)
 			(do_not_autoplace no)
@@
 		)
 		(property "Footprint" "TerminalBlock_Phoenix:TerminalBlock_Phoenix_MKDS-1,5-2_1x02_P5.00mm_Horizontal"
-			(at 40.64 38.1 0)
+			(at 27.94 38.1 0)
 			(hide yes)
 			(show_name no)
@@
 		)
 		(property "Datasheet" ""
-			(at 40.64 38.1 0)
+			(at 27.94 38.1 0)
 			(hide yes)
 			(show_name no)
@@
 		)
 		(property "Description" "Generic screw terminal, single row, 01x02, script generated (kicad-library-utils/schlib/autogen/connector/)"
-			(at 40.64 38.1 0)
+			(at 27.94 38.1 0)
 			(hide yes)
 			(show_name no)

Commit message: sensor iteration 2
Parts:
- removed R9: 0R, Resistor_SMD:R_2512_6332Metric_Pad1.40x3.35mm_HandSolder, symbol Device:R
- added R13: 0R, Resistor_SMD:R_2512_6332Metric_Pad1.40x3.35mm_HandSolder, symbol Device:R
Connections:
- net LORA_DIO0: now also U2.5 (DIO0)
- net LORA_RESET: now also R13.1; no longer U2.4 (~{RESET})
- new net: R13.2, U2.4 (~{RESET})
Other:
- moved on the sheet: R8
Changed lines of the file:
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@@
+	)
+	(junction
+		(at 64.77 157.48)
+		(diameter 0)
+		(color 0 0 0 0)
 	)
 	(junction
@@
 		(color 0 0 0 0)
 	)
-	(junction
-		(at 81.28 157.48)
-		(diameter 0)
-		(color 0 0 0 0)
-	)
 	(no_connect
 		(at 123.19 154.94)
@@
 	(wire
 		(pts
-			(xy 123.19 149.86) (xy 127 149.86)
+			(xy 123.19 149.86) (xy 137.16 149.86)
 		)
 		(stroke
@@
 	(wire
 		(pts
-			(xy 60.96 157.48) (xy 81.28 157.48)
+			(xy 52.07 157.48) (xy 64.77 157.48)
 		)
 		(stroke
@@
 	(wire
 		(pts
-			(xy 81.28 173.99) (xy 74.93 173.99)
+			(xy 64.77 173.99) (xy 58.42 173.99)
 		)
 		(stroke
@@
 	(wire
 		(pts
-			(xy 134.62 149.86) (xy 149.86 149.86)
-		)
-		(stroke
-			(width 0)
-			(type default)
-		)
-	)
-	(wire
-		(pts
 			(xy 143.51 82.55) (xy 130.81 82.55)
 		)
@@
 	(wire
 		(pts
-			(xy 81.28 157.48) (xy 102.87 157.48)
-		)
-		(stroke
-			(width 0)
-			(type default)
-		)
-	)
-	(wire
-		(pts
-			(xy 81.28 170.18) (xy 81.28 173.99)
+			(xy 64.77 157.48) (xy 102.87 157.48)
+		)
+		(stroke
+			(width 0)
+			(type default)
+		)
+	)
+	(wire
+		(pts
+			(xy 64.77 170.18) (xy 64.77 173.99)
 		)
 		(stroke
@@
 	(wire
 		(pts
-			(xy 90.17 162.56) (xy 102.87 162.56)
+			(xy 77.47 162.56) (xy 92.71 162.56)
 		)
 		(stroke
@@
 	(wire
 		(pts
-			(xy 81.28 157.48) (xy 81.28 162.56)
+			(xy 64.77 157.48) (xy 64.77 162.56)
 		)
 		(stroke
@@
 		(pts
 			(xy 168.91 19.05) (xy 170.18 19.05)
+		)
+		(stroke
+			(width 0)
+			(type default)
+		)
+	)
+	(wire
+		(pts
+			(xy 100.33 162.56) (xy 102.87 162.56)
 		)
 		(stroke
@@
 	)
 	(label "LORA_NSS"
-		(at 60.96 157.48 0)
+		(at 52.07 157.48 0)
 		(effects
 			(font
@@
 	)
 	(label "LORA_DIO0"
-		(at 149.86 149.86 180)
+		(at 137.16 149.86 180)
 		(effects
 			(font
@@
 	)
 	(label "LORA_RESET"
-		(at 90.17 162.56 0)
+		(at 77.47 162.56 0)
 		(effects
 			(font
@@
 			)
 			(justify left bottom)
+		)
+	)
+	(netclass_flag ""
+		(length 2.54)
+		(shape round)
+		(at 34.29 38.1 0)
+		(fields_autoplaced yes)
+		(effects
+			(font
+				(size 1.27 1.27)
+			)
+			(justify left bottom)
+		)
+		(property "Netclass" "Power 220V0"
+			(at 34.9885 35.56 0)
+			(show_name no)
+			(do_not_autoplace no)
+			(effects
+				(font
+					(size 1.27 1.27)
+				)
+				(justify left)
+			)
+		)
+		(property "Component Class" ""
+			(at -41.91 8.89 0)
+			(show_name no)
+			(do_not_autoplace no)
+			(effects
+				(font
+					(size 1.27 1.27)
+					(italic yes)
+				)
+			)
 		)
 	)
@@
 	)
 	(symbol
-		(lib_id "Device:R")
-		(at 130.81 149.86 90)
-		(unit 1)
-		(body_style 1)
-		(exclude_from_sim no)
-		(in_bom yes)
-		(on_board yes)
-		(in_pos_files yes)
-		(dnp no)
-		(fields_autoplaced yes)
-		(property "Reference" "R9"
-			(at 130.81 143.51 90)
-			(show_name no)
-			(do_not_autoplace no)
-			(effects
-				(font
-					(size 1.27 1.27)
-				)
-			)
-		)
-		(property "Value" "0R"
-			(at 130.81 146.05 90)
-			(show_name no)
-			(do_not_autoplace no)
-			(effects
-				(font
-					(size 1.27 1.27)
-				)
-			)
-		)
-		(property "Footprint" "Resistor_SMD:R_2512_6332Metric_Pad1.40x3.35mm_HandSolder"
-			(at 130.81 151.638 90)
-			(hide yes)
-			(show_name no)
-			(do_not_autoplace no)
-			(effects
-				(font
-					(size 1.27 1.27)
-				)
-			)
-		)
-		(property "Datasheet" ""
-			(at 130.81 149.86 0)
-			(hide yes)
-			(show_name no)
-			(do_not_autoplace no)
-			(effects
-				(font
-					(size 1.27 1.27)
-				)
-			)
-		)
-		(property "Description" "Resistor"
-			(at 130.81 149.86 0)
-			(hide yes)
-			(show_name no)
-			(do_not_autoplace no)
-			(effects
-				(font
-					(size 1.27 1.27)
-				)
-			)
-		)
-		(pin "1"
-		)
-		(pin "2"
-		)
-		(instances
-			(project "active_sender"
-				(path "/0a63acd0-8ffb-408e-b0ed-0179bed06f72"
-					(reference "R9")
-					(unit 1)
-				)
-			)
-		)
-	)
-	(symbol
 		(lib_id "power:+3.3V")
 		(at 113.03 132.08 0)
@@
 	(symbol
 		(lib_id "power:+3.3V")
-		(at 74.93 173.99 0)
+		(at 58.42 173.99 0)
 		(unit 1)
 		(body_style 1)
@@
 		(fields_autoplaced yes)
 		(property "Reference" "#PWR017"
-			(at 74.93 177.8 0)
+			(at 58.42 177.8 0)
 			(hide yes)
 			(show_name no)
@@
 		)
 		(property "Value" "+3.3V"
-			(at 74.93 168.91 0)
+			(at 58.42 168.91 0)
 			(show_name no)
 			(do_not_autoplace no)
@@
 		)
 		(property "Footprint" ""
-			(at 74.93 173.99 0)
+			(at 58.42 173.99 0)
 			(hide yes)
 			(show_name no)
@@
 		)
 		(property "Datasheet" ""
-			(at 74.93 173.99 0)
+			(at 58.42 173.99 0)
 			(hide yes)
 			(show_name no)
@@
 		)
 		(property "Description" "Power symbol creates a global label with name \"+3.3V\""
-			(at 74.93 173.99 0)
+			(at 58.42 173.99 0)
 			(hide yes)
 			(show_name no)
@@
 	(symbol
 		(lib_id "Device:R")
-		(at 81.28 166.37 0)
+		(at 64.77 166.37 0)
 		(unit 1)
 		(body_style 1)
@@
 		(fields_autoplaced yes)
 		(property "Reference" "R8"
-			(at 83.82 165.0999 0)
+			(at 67.31 165.0999 0)
 			(show_name no)
 			(do_not_autoplace no)
@@
 		)
 		(property "Value" "10k"
-			(at 83.82 167.6399 0)
+			(at 67.31 167.6399 0)
 			(show_name no)
 			(do_not_autoplace no)
@@
 		)
 		(property "Footprint" "Resistor_SMD:R_1206_3216Metric_Pad1.30x1.75mm_HandSolder"
-			(at 79.502 166.37 90)
+			(at 62.992 166.37 90)
 			(hide yes)
 			(show_name no)
@@
 		)
 		(property "Datasheet" ""
-			(at 81.28 166.37 0)
+			(at 64.77 166.37 0)
 			(hide yes)
 			(show_name no)
@@
 		)
 		(property "Description" "Resistor"
-			(at 81.28 166.37 0)
+			(at 64.77 166.37 0)
 			(hide yes)
 			(show_name no)
@@
 					(unit 1)
 				)
+			)
+		)
+	)
+	(symbol
+		(lib_id "Device:R")
+		(at 96.52 162.56 90)
+		(mirror x)
+		(unit 1)
+		(body_style 1)
+		(exclude_from_sim no)
+		(in_bom yes)
+		(on_board yes)
+		(in_pos_files yes)
+		(dnp no)
+		(property "Reference" "R13"
+			(at 96.52 158.242 90)
+			(show_name no)
+			(do_not_autoplace no)
+			(effects
+				(font
+					(size 1.27 1.27)
+				)
+			)
+		)
+		(property "Value" "0R"
+			(at 96.52 160.274 90)
+			(show_name no)
+			(do_not_autoplace no)
+			(effects
+				(font
+					(size 1.27 1.27)
+				)
+			)
+		)
+		(property "Footprint" "Resistor_SMD:R_2512_6332Metric_Pad1.40x3.35mm_HandSolder"
+			(at 96.52 160.782 90)
+			(hide yes)
+			(show_name no)
+			(do_not_autoplace no)
+			(effects
+				(font
+					(size 1.27 1.27)
+				)
+			)
+		)
+		(property "Datasheet" ""
+			(at 96.52 162.56 0)
+			(hide yes)
+			(show_name no)
+			(do_not_autoplace no)
+			(effects
+				(font
+					(size 1.27 1.27)
+				)
+			)
+		)
+		(property "Description" "Resistor"
+			(at 96.52 162.56 0)
+			(hide yes)
+			(show_name no)
+			(do_not_autoplace no)
+			(effects
+				(font
+					(size 1.27 1.27)
+				)
+			)
+		)
+		(pin "1"
+		)
+		(pin "2"
+		)
+		(instances
+			(project "active_sender"
+				(path "/0a63acd0-8ffb-408e-b0ed-0179bed06f72"
+					(reference "R13")
+					(unit 1)
+				)

Commit message: sensor iteration 3
Parts:
- added R5: 10k, Resistor_SMD:R_1206_3216Metric_Pad1.30x1.75mm_HandSolder, symbol Device:R
- added R9: 330, Resistor_SMD:R_1206_3216Metric_Pad1.30x1.75mm_HandSolder, symbol Device:R
Connections:
- net GNDPWR: now also R5.2
- net at R6.1: now also R9.2; no longer Q1.1 (G)
- new net: Q1.1 (G), R5.1, R9.1
Other:
- moved on the sheet: D1, J2, Q1
