File: hardware/gateway/KiCAD/gateway.kicad_pcb (KiCad board)
At the start: 2 copper layers, 88 x 74 mm, 29 parts, among them J1 USB-C input, J2 Buzzer, J3 Water Sensor, Q1 AO3400A, SW1 SW_Push, SW2 SW_SPDT, U1 ESP32-C3_SUPERMINI_TH, U2 Ai-Thinker-Ra-02, U3 AMS1117-3.3

Commit message: dev
Parts:
- removed C2: 470u, Capacitor_THT:C_Radial_D8.0mm_H11.5mm_P3.50mm
- removed D1: SS34, Diode_SMD:D_SMA
- removed J2: Buzzer, TerminalBlock_Phoenix:TerminalBlock_Phoenix_MKDS-1,5-2_1x02_P5.00mm_Horizontal
- removed J3: Water Sensor, Connector_JST:JST_XH_S4B-XH-A-1_1x04_P2.50mm_Horizontal
- removed R1: 10k, Resistor_SMD:R_1206_3216Metric_Pad1.30x1.75mm_HandSolder
- removed R2: 3.9k, Resistor_SMD:R_1206_3216Metric_Pad1.30x1.75mm_HandSolder
- removed R6: 0R, Resistor_SMD:R_2512_6332Metric_Pad1.40x3.35mm_HandSolder
- removed REF** (x4): MountingHole_2.2mm_M2_DIN965_Pad_TopOnly, MountingHole:MountingHole_2.2mm_M2_DIN965_Pad_TopOnly
- removed SW1: SW_Push, Button_Switch_THT:SW_PUSH_6mm_H5mm
- removed SW2: SW_SPDT, custom_footprints:SS12D00
- added BTN1: SW_Push, Button_Switch_THT:SW_PUSH_6mm_H5mm, F.Cu at (61.8, 58.8)
- added BTN2: SW_Push, Button_Switch_THT:SW_PUSH_6mm_H5mm, F.Cu at (61.8, 73.8)
- added BTN3: SW_Push, Button_Switch_THT:SW_PUSH_6mm_H5mm, F.Cu at (61.8, 88.8)
- added BTN4: SW_Push, Button_Switch_THT:SW_PUSH_6mm_H5mm, F.Cu at (61.8, 103.8)
- added BTN5: SW_Push, Button_Switch_THT:SW_PUSH_6mm_H5mm, F.Cu at (61.8, 118.8)
- added BZ1: Buzzer, Buzzer_Beeper:Buzzer_12x9.5RM7.6, F.Cu at (85.0, 71.0)
- added LED1: APA-106-F5, LED_THT:LED_D5.0mm-4_RGB_Staggered_Pins, F.Cu at (77.0, 63.4)
- added LED2: APA-106-F5, LED_THT:LED_D5.0mm-4_RGB_Staggered_Pins, F.Cu at (77.0, 78.4)
- added LED3: APA-106-F5, LED_THT:LED_D5.0mm-4_RGB_Staggered_Pins, F.Cu at (77.0, 93.4)
- added LED4: APA-106-F5, LED_THT:LED_D5.0mm-4_RGB_Staggered_Pins, F.Cu at (77.0, 108.4)
- added LED5: APA-106-F5, LED_THT:LED_D5.0mm-4_RGB_Staggered_Pins, F.Cu at (77.0, 123.4)
- added R14: 15k,0603, Resistor_SMD:R_0805_2012Metric_Pad1.20x1.40mm_HandSolder, B.Cu at (65.0, 114.0)
- added R15: 330,0603, Resistor_SMD:R_0805_2012Metric_Pad1.20x1.40mm_HandSolder, B.Cu at (93.0, 63.0)
- added R16: 100,0603, Resistor_SMD:R_0805_2012Metric_Pad1.20x1.40mm_HandSolder, B.Cu at (86.0, 79.0)
- C1: value 104 0.1uF -> 0.1u
- R10: value 0R -> 6.8k,0603; footprint Resistor_SMD:R_2512_6332Metric_Pad1.40x3.35mm_HandSolder -> Resistor_SMD:R_0805_2012Metric_Pad1.20x1.40mm_HandSolder
- R3, R5, R8, R9: footprint Resistor_SMD:R_1206_3216Metric_Pad1.30x1.75mm_HandSolder -> Resistor_SMD:R_0805_2012Metric_Pad1.20x1.40mm_HandSolder
- R4: value 330 -> 2.2k,0603; footprint Resistor_SMD:R_1206_3216Metric_Pad1.30x1.75mm_HandSolder -> Resistor_SMD:R_0805_2012Metric_Pad1.20x1.40mm_HandSolder
- R7: value 0R -> 3.3k,0603; footprint Resistor_SMD:R_2512_6332Metric_Pad1.40x3.35mm_HandSolder -> Resistor_SMD:R_0805_2012Metric_Pad1.20x1.40mm_HandSolder
- moved R4 71.4 mm to (65.0, 68.0), turned to -90 degrees
- moved R7 52.5 mm to (65.0, 83.0), turned to -90 degrees
- moved R9 43.0 mm to (89.0, 86.0), turned to -90 degrees
- moved R12 41.7 mm to (86.0, 57.0), turned to 180 degrees
- moved R5 40.8 mm to (85.0, 86.0), turned to -90 degrees
- moved R11 36.1 mm to (95.0, 57.0)
- moved R10 33.8 mm to (65.0, 98.0)
- moved C1 30.1 mm to (82.0, 98.0), turned to -90 degrees
- moved R3 30.1 mm to (86.0, 98.0)
- moved Q1 26.6 mm to (79.8, 84.0)
- moved U3 24.0 mm to (90.7, 107.8)
- moved J1 20.0 mm to (93.0, 122.0), turned to 180 degrees
- moved U2 20.0 mm to (110.9, 72.3)
- moved R13 20.0 mm to (107.9, 68.3), turned to -90 degrees
- moved R8 20.0 mm to (116.9, 75.3)
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Connections:
- C1 pad 1: /LINK_BUTTON -> /LINK_BUTTONS
- J1 pad 1: Net-(J1-Pin_1) -> +5V
- Q1 pad 2: GNDPWR -> GNDD
- R10 pad 1: Net-(SW2-B) -> Net-(BTN3-Pad2)
- R10 pad 2: /MODE -> Net-(BTN4-Pad2)
- R13 pad 1: /LORA_RESET -> Net-(U2-~{RESET})
- R13 pad 2: Net-(U2-~{RESET}) -> /LORA_RESET
- R3 pad 1: +3.3V -> /LINK_BUTTONS
- R3 pad 2: /LINK_BUTTON -> /+3V0 MCU
- R4 pad 1: /LINK_BUTTON -> /LINK_BUTTONS
- R4 pad 2: Net-(R4-Pad2) -> Net-(BTN2-Pad2)
- R5 pad 2: GNDPWR -> GNDD
- R7 pad 1: /SENSOR -> Net-(BTN2-Pad2)
- R7 pad 2: Net-(R1-Pad2) -> Net-(BTN3-Pad2)
- R8 pad 2: +3.3V -> Net-(U2-VDD)
- R9 pad 2: Net-(R6-Pad1) -> /BUZZER
- U1 pad 1: /SENSOR -> /LINK_BUTTONS
- U1 pad 2: unconnected-(U1-GPIO2-Pad2) -> /LED_LINE
- U1 pad 3.3: +3.3V -> /+3V0 MCU
- U1 pad 5V: unconnected-(U1-Pad5V) -> +5V
- U1 pad 9: /LINK_BUTTON -> unconnected-(U1-GPIO9-Pad9)
- U2 pad 3: +3.3V -> Net-(U2-VDD)
- U3 pad 2: +3.3V -> Net-(U2-VDD)
- U3 pad 3: Net-(J1-Pin_1) -> +5V
Routing:
- net /12V0: track 92.9 -> 0.00 mm
- net +3.3V: track 90.4 -> 0.00 mm
- net /LINK_BUTTON: track 53.9 -> 0.00 mm
- net Net-(R4-Pad2): track 50.6 -> 0.00 mm
- net GNDD: track 38.3 -> 0.00 mm
- net Net-(U2-VDD): track 0.00 -> 30.2 mm
- net Net-(J3-Pin_2): track 25.5 -> 0.00 mm
- net Net-(J1-Pin_1): track 16.6 -> 0.00 mm
- net Net-(Q1-G): track 16.2 -> 0.00 mm
- net Net-(R1-Pad2): track 12.1 -> 0.00 mm
- net Net-(BZ1--): track 11.9 -> 0.00 mm
- net /BUZZER: track 8.41 -> 0.00 mm
- net /SENSOR: track 6.94 -> 0.00 mm
- net /MODE: track 6.57 -> 0.00 mm
- net Net-(SW2-B): track 6.43 -> 0.00 mm
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Other:
- board size 88 x 74 mm -> 70 x 74 mm

Commit message: dev
Parts:
- added R17: 0R, Resistor_SMD:R_2512_6332Metric_Pad1.40x3.35mm_HandSolder, B.Cu at (88.0, 89.5)
- added R18: 0R, Resistor_SMD:R_2512_6332Metric_Pad1.40x3.35mm_HandSolder, B.Cu at (95.5, 113.5)
- R10: value 6.8k,0603 -> 6.8k,0805
- R14: value 15k,0603 -> 15k,0805
- R15: value 330,0603 -> 330,0805
- R16: value 100,0603 -> 100,0805
- R3: value 10k,0603 -> 10k,0805
- R4: value 2.2k,0603 -> 2.2k,0805
- R5, R8: value 10k -> 10k,0805
- R7: value 3.3k,0603 -> 3.3k,0805
- R9: value 330 -> 330,0805
- moved R12 63.0 mm to (87.5, 120.0)
- moved J1 41.8 mm to (88.0, 80.5), turned to 0 degrees
- moved U3 39.9 mm to (90.5, 68.0)
- moved BZ1 38.0 mm to (84.0, 109.0)
- moved R16 25.1 mm to (84.0, 104.0), turned to 90 degrees
- moved Q1 24.3 mm to (92.0, 105.0), turned to -90 degrees
- moved R11 18.4 mm to (99.0, 75.0)
- moved C1 17.8 mm to (99.5, 94.5), turned to 90 degrees
- moved R3 15.2 mm to (99.5, 105.0)
- moved R5 13.9 mm to (91.0, 98.5), turned to 90 degrees
- moved R9 13.7 mm to (94.5, 98.5), turned to 90 degrees
- moved R15 11.4 mm to (83.0, 68.5), turned to -90 degrees
- moved R4 2.00 mm to (67.0, 68.0), turned to 180 degrees
- moved R14 1.00 mm to (65.0, 113.0), turned to 0 degrees
- moved R8 0.12 mm to (117.0, 75.3)
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Connections:
- R15 pad 2: /LED_LINE -> Net-(R15-Pad2)
- U1 pad 5V: +5V -> Net-(R18-Pad2)
Routing:
- net +5V: track 0.00 -> 154.8 mm
- net /LINK_BUTTONS: track 0.00 -> 130.6 mm
- net /LED_LINE: track 0.00 -> 27.2 mm
- net Net-(BTN4-Pad2): track 0.00 -> 23.4 mm
- net Net-(BTN3-Pad2): track 0.00 -> 23.4 mm
- net Net-(BTN2-Pad2): track 0.00 -> 23.4 mm
- net Net-(R15-Pad2): track 0.00 -> 20.8 mm
- net Net-(BTN5-Pad2): track 0.00 -> 17.7 mm
- net Net-(U2-VDD): track 30.2 -> 46.9 mm
- net /BUZZER: track 0.00 -> 16.0 mm
- net Net-(LED1-DI): track 0.00 -> 12.6 mm
- net Net-(LED4-DO): track 0.00 -> 10.8 mm
- net Net-(LED3-DO): track 0.00 -> 10.8 mm
- net Net-(LED2-DO): track 0.00 -> 10.8 mm
- net Net-(LED1-DO): track 0.00 -> 10.8 mm
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
Commit message: dev
Parts:
- removed R18: 0R, Resistor_SMD:R_2512_6332Metric_Pad1.40x3.35mm_HandSolder
- added R19: 0R, Resistor_SMD:R_2512_6332Metric_Pad1.40x3.35mm_HandSolder, B.Cu at (95.5, 87.5)
- added R20: 0R, Resistor_SMD:R_2512_6332Metric_Pad1.40x3.35mm_HandSolder, B.Cu at (88.0, 93.5)
- added R21: 0R, Resistor_SMD:R_2512_6332Metric_Pad1.40x3.35mm_HandSolder, B.Cu at (76.2, 69.5)
- added R22: 0R, Resistor_SMD:R_2512_6332Metric_Pad1.40x3.35mm_HandSolder, B.Cu at (96.0, 115.0)
- added REF**: MountingHole_2.2mm_M2_DIN965_Pad_TopOnly, MountingHole:MountingHole_2.2mm_M2_DIN965_Pad_TopOnly, B.Cu at (91.0, 124.0)
- added REF**: MountingHole_2.2mm_M2_DIN965_Pad_TopOnly, MountingHole:MountingHole_2.2mm_M2_DIN965_Pad_TopOnly, B.Cu at (91.0, 59.0)
- moved R12 54.7 mm to (115.2, 72.8), turned to 45 degrees
- moved R16 8.54 mm to (87.0, 112.0), turned to 180 degrees
- moved R15 7.32 mm to (84.0, 75.8)
- moved R8 4.19 mm to (117.0, 79.5)
- moved BZ1 4.12 mm to (88.0, 108.0)
- moved Q1 3.35 mm to (95.0, 103.5)
- moved C1 3.04 mm to (100.0, 97.5), turned to 180 degrees
- moved R4 2.06 mm to (65.0, 68.5), turned to -90 degrees
- moved R17 1.50 mm to (88.0, 88.0)
- moved R3 1.50 mm to (101.0, 105.0)
- moved R14 1.00 mm to (65.0, 114.0), turned to -90 degrees
- moved BTN1 0.50 mm to (61.8, 59.2)
- moved BTN2 0.50 mm to (61.8, 74.2)
- moved BTN3 0.50 mm to (61.8, 89.2)
- moved BTN4 0.50 mm to (61.8, 104.2)
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Connections:
- BTN1 pad 2: /LINK_BUTTONS -> Net-(BTN1-Pad2)
- R4 pad 1: /LINK_BUTTONS -> Net-(BTN1-Pad2)
- U1 pad 5V: Net-(R18-Pad2) -> +5V
Routing:
- net Net-(BTN1-Pad2): track 0.00 -> 116.0 mm
- net /LINK_BUTTONS: track 130.6 -> 23.2 mm
- net +5V: track 154.8 -> 175.3 mm
- net Net-(R15-Pad2): track 20.8 -> 11.6 mm
- net Net-(R18-Pad2): track 7.43 -> 0.00 mm
- net Net-(LED1-DI): track 12.6 -> 19.7 mm
- net /LORA_NSS: track 32.5 -> 27.4 mm
- net Net-(U2-VDD): track 46.9 -> 51.0 mm
- net /BUZZER: track 16.0 -> 12.2 mm
- net Net-(BTN3-Pad2): track 23.4 -> 19.5 mm
- net Net-(BTN2-Pad2): track 23.4 -> 19.5 mm
- net Net-(BTN4-Pad2): track 23.4 -> 20.0 mm
- net Net-(BTN5-Pad2): track 17.7 -> 15.2 mm
- net /+3V0 MCU: track 5.42 -> 3.92 mm
- net Net-(U2-~{RESET}): track 7.94 -> 9.38 mm
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Other:
- board size 70 x 74 mm -> 70 x 75 mm

Commit message: dev
Parts:
- R16: value 100,0805 -> 330,0805
