File: hardware/sensor/KiCAD/active_sender.kicad_sch (KiCad schematic)
At the start: 27 parts, among them J1 220V0, J2 Buzzer, J3 Water Sensor, Q1 AO3400A, SW1 SW_Push, SW2 SW_SPDT, U1 ESP32-C3_SUPERMINI_TH, U2 Ai-Thinker-Ra-02, U3 HLK-PM12

Commit message: dev
Parts:
- R2: value 3.9k -> 10k
Changed lines of the file:
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@@
 			)
 		)
-		(property "Value" "3.9k"
+		(property "Value" "10k"
 			(at 75.184 92.71 0)
 			(show_name no)

Commit message: dev
Parts:
- removed DC1: Mini 560 Step-down 12V0->3V3, custom_footprints:MINI 560 PRO, symbol Custom_library:Mini 560 Step-down
- removed F1: Fuse, Fuse:Fuseholder_Cylinder-5x20mm_Schurter_0031_8201_Horizontal_Open, symbol Device:Fuse
- removed R11, R12: 0R, Resistor_SMD:R_2512_6332Metric_Pad1.40x3.35mm_HandSolder, symbol Device:R
- removed U3: HLK-PM12, Converter_ACDC:Converter_ACDC_Hi-Link_HLK-PMxx, symbol Converter_ACDC:HLK-PM12
- added U3: AMS1117-3.3, Package_TO_SOT_SMD:SOT-223-3_TabPin2, symbol Regulator_Linear:AMS1117-3.3
- added U4: (no value), custom_footprints:CKCS BS-01, symbol Custom_library:CKCS_BS-01
- C2: value 470u -> 100-220uF; footprint Capacitor_THT:C_Radial_D8.0mm_H11.5mm_P3.50mm -> Capacitor_SMD:C_Elec_5x5.4
- J1: value 220V0 -> USB-C input
Connections:
- net N 220V0 is gone; now on net GNDD: J1.2 (Pin_2)
- net +3.3V: now also C2.2, R2.2, U3.2 (VO)
- net GNDD: now also C2.1, J3.3 (Pin_3), Q1.2 (S), R5.2, SW2.1 (A), U3.1 (GND), U4.2 (IN-), U4.4 (OUT-); no longer R2.2
- net +5V: now reaches J1.1 (Pin_1)
- net +5V: now also J3.1 (Pin_1), SW2.3 (C), U3.3 (VI), U4.1 (IN+)
- removed net 12V0: C2.1, D1.1 (K), J2.2 (Pin_2), J3.1 (Pin_1), SW2.3 (C)
- removed net GNDPWR: C2.2, J3.3 (Pin_3), Q1.2 (S), R5.2, SW2.1 (A)
- new net +12V: D1.1 (K), J2.2 (Pin_2), U4.3 (OUT+)
Other:
- moved on the sheet: D1, J2, J3, R13, R8, U2

Commit message: dev
Parts:
- R2, R5, R8: value 10k -> 10k,1206
- R3: value 10k,0603 -> 10k,1206
- R4, R9: value 330 -> 330,1206
Other:
- moved on the sheet: R5
Changed lines of the file:
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@@
 	(paper "A4" portrait)
 	(junction
-		(at 69.85 60.96)
+		(at 125.73 160.02)
 		(diameter 0)
 		(color 0 0 0 0)
 	)
 	(junction
-		(at 125.73 160.02)
+		(at 69.85 60.96)
 		(diameter 0)
 		(color 0 0 0 0)
@@
 	)
 	(junction
-		(at 60.96 69.85)
-		(diameter 0)
-		(color 0 0 0 0)
-	)
-	(junction
 		(at 62.23 29.21)
 		(diameter 0)
@@
 	)
 	(junction
+		(at 60.96 71.12)
+		(diameter 0)
+		(color 0 0 0 0)
+	)
+	(junction
 		(at 71.12 85.09)
 		(diameter 0)
@@
 	(wire
 		(pts
-			(xy 69.85 60.96) (xy 78.74 60.96)
+			(xy 69.85 60.96) (xy 83.82 60.96)
 		)
 		(stroke
@@
 	(wire
 		(pts
+			(xy 60.96 68.58) (xy 60.96 71.12)
+		)
+		(stroke
+			(width 0)
+			(type default)
+		)
+	)
+	(wire
+		(pts
 			(xy 102.87 176.53) (xy 115.57 176.53)
 		)
@@
 	(wire
 		(pts
-			(xy 60.96 69.85) (xy 69.85 69.85)
+			(xy 60.96 71.12) (xy 69.85 71.12)
 		)
 		(stroke
@@
 	(wire
 		(pts
-			(xy 78.74 60.96) (xy 78.74 67.31)
+			(xy 83.82 60.96) (xy 83.82 67.31)
 		)
 		(stroke
@@
 	(wire
 		(pts
+			(xy 69.85 62.23) (xy 69.85 60.96)
+		)
+		(stroke
+			(width 0)
+			(type default)
+		)
+	)
+	(wire
+		(pts
 			(xy 40.64 106.68) (xy 31.75 106.68)
 		)
@@
 	(wire
 		(pts
-			(xy 60.96 72.39) (xy 60.96 69.85)
+			(xy 60.96 72.39) (xy 60.96 71.12)
 		)
 		(stroke
@@
 	(wire
 		(pts
-			(xy 60.96 69.85) (xy 60.96 68.58)
+			(xy 69.85 71.12) (xy 69.85 69.85)
 		)
 		(stroke
@@
 	(wire
 		(pts
-			(xy 69.85 68.58) (xy 69.85 69.85)
-		)
-		(stroke
-			(width 0)
-			(type default)
-		)
-	)
-	(wire
-		(pts
 			(xy 100.33 26.67) (xy 110.49 26.67)
 		)
@@
 			)
 		)
-		(property "Value" "10k"
+		(property "Value" "10k,1206"
 			(at 80.01 194.3099 0)
 			(show_name no)
@@
 			)
 		)
-		(property "Value" "10k"
+		(property "Value" "10k,1206"
 			(at 75.184 92.71 0)
 			(show_name no)
@@
 			)
 		)
-		(property "Value" "330"
+		(property "Value" "330,1206"
 			(at 163.83 83.82 90)
 			(show_name no)
@@
 			)
 		)
-		(property "Value" "330"
+		(property "Value" "330,1206"
 			(at 63.5 77.4699 0)
 			(show_name no)
@@
 			)
 		)
-		(property "Value" "10k,0603"
+		(property "Value" "10k,1206"
 			(at 154.94 82.5499 0)
 			(show_name no)
@@
 	(symbol
 		(lib_id "power:GNDD")
-		(at 78.74 67.31 0)
+		(at 83.82 67.31 0)
 		(unit 1)
 		(body_style 1)
@@
 		(fields_autoplaced yes)
 		(property "Reference" "#PWR09"
-			(at 78.74 73.66 0)
+			(at 83.82 73.66 0)
 			(hide yes)
 			(show_name no)
@@
 		)
 		(property "Value" "GNDD"
-			(at 78.74 71.12 0)
+			(at 83.82 71.12 0)
 			(show_name no)
 			(do_not_autoplace no)
@@
 		)
 		(property "Footprint" ""
-			(at 78.74 67.31 0)
+			(at 83.82 67.31 0)
 			(hide yes)
 			(show_name no)
@@
 		)
 		(property "Datasheet" ""
-			(at 78.74 67.31 0)
+			(at 83.82 67.31 0)
 			(hide yes)
 			(show_name no)
@@
 		)
 		(property "Description" "Power symbol creates a global label with name \"GNDD\" , digital ground"
-			(at 78.74 67.31 0)
+			(at 83.82 67.31 0)
 			(hide yes)
 			(show_name no)
@@
 	(symbol
 		(lib_id "Device:R")
-		(at 69.85 64.77 180)
+		(at 69.85 66.04 180)
 		(unit 1)
 		(body_style 1)
@@
 		(fields_autoplaced yes)
 		(property "Reference" "R5"
-			(at 72.39 63.4999 0)
+			(at 72.39 64.7699 0)
 			(show_name no)
 			(do_not_autoplace no)
@@
 			)
 		)
-		(property "Value" "10k"
-			(at 72.39 66.0399 0)
+		(property "Value" "10k,1206"
+			(at 72.39 67.3099 0)
 			(show_name no)
 			(do_not_autoplace no)
@@
 		)
 		(property "Footprint" "Resistor_SMD:R_1206_3216Metric_Pad1.30x1.75mm_HandSolder"
-			(at 71.628 64.77 90)
+			(at 71.628 66.04 90)
 			(hide yes)
 			(show_name no)
@@
 		)
 		(property "Datasheet" ""
-			(at 69.85 64.77 0)
+			(at 69.85 66.04 0)
 			(hide yes)
 			(show_name no)
@@
 		)
 		(property "Description" "Resistor"
-			(at 69.85 64.77 0)
+			(at 69.85 66.04 0)
 			(hide yes)
 			(show_name no)

Commit message: dev
Connections:
- net +5V: now also U4.2 (IN+); no longer U4.1 (IN+)
- net GNDD: now also U4.1 (IN-); no longer U4.2 (IN-)
Changed lines of the file:
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@@
+	)
+	(junction
+		(at 62.23 26.67)
+		(diameter 0)
+		(color 0 0 0 0)
+	)
+	(junction
+		(at 157.48 87.63)
+		(diameter 0)
+		(color 0 0 0 0)
+	)
+	(junction
+		(at 46.99 60.96)
+		(diameter 0)
+		(color 0 0 0 0)
 	)
 	(junction
@@
 	)
 	(junction
-		(at 157.48 87.63)
-		(diameter 0)
-		(color 0 0 0 0)
-	)
-	(junction
-		(at 46.99 60.96)
-		(diameter 0)
-		(color 0 0 0 0)
-	)
-	(junction
-		(at 62.23 26.67)
+		(at 62.23 30.48)
 		(diameter 0)
 		(color 0 0 0 0)
@@
 	(wire
 		(pts
+			(xy 62.23 29.21) (xy 69.85 29.21)
+		)
+		(stroke
+			(width 0)
+			(type default)
+		)
+	)
+	(wire
+		(pts
 			(xy 60.96 71.12) (xy 69.85 71.12)
 		)
@@
 	(wire
 		(pts
+			(xy 62.23 30.48) (xy 62.23 31.75)
+		)
+		(stroke
+			(width 0)
+			(type default)
+		)
+	)
+	(wire
+		(pts
+			(xy 76.2 29.21) (xy 80.01 29.21)
+		)
+		(stroke
+			(width 0)
+			(type default)
+		)
+	)
+	(wire
+		(pts
 			(xy 60.96 85.09) (xy 60.96 104.14)
 		)
@@
 	(wire
 		(pts
-			(xy 62.23 30.48) (xy 62.23 29.21)
-		)
-		(stroke
-			(width 0)
-			(type default)
-		)
-	)
-	(wire
-		(pts
 			(xy 45.72 101.6) (xy 45.72 110.49)
 		)
@@
 	(wire
 		(pts
+			(xy 67.31 24.13) (xy 76.2 24.13)
+		)
+		(stroke
+			(width 0)
+			(type default)
+		)
+	)
+	(wire
+		(pts
 			(xy 143.51 77.47) (xy 130.81 77.47)
 		)
@@
 	(wire
 		(pts
+			(xy 62.23 22.86) (xy 62.23 26.67)
+		)
+		(stroke
+			(width 0)
+			(type default)
+		)
+	)
+	(wire
+		(pts
 			(xy 90.17 189.23) (xy 105.41 189.23)
 		)
@@
 	(wire
 		(pts
+			(xy 69.85 29.21) (xy 69.85 26.67)
+		)
+		(stroke
+			(width 0)
+			(type default)
+		)
+	)
+	(wire
+		(pts
 			(xy 40.64 106.68) (xy 31.75 106.68)
 		)
@@
 	(wire
 		(pts
-			(xy 62.23 26.67) (xy 52.07 26.67)
+			(xy 52.07 26.67) (xy 62.23 26.67)
 		)
 		(stroke
@@
 	(wire
 		(pts
-			(xy 62.23 22.86) (xy 62.23 26.67)
-		)
-		(stroke
-			(width 0)
-			(type default)
-		)
-	)
-	(wire
-		(pts
 			(xy 157.48 97.79) (xy 157.48 100.33)
 		)
@@
 	(wire
 		(pts
+			(xy 62.23 29.21) (xy 62.23 30.48)
+		)
+		(stroke
+			(width 0)
+			(type default)
+		)
+	)
+	(wire
+		(pts
 			(xy 53.34 99.06) (xy 55.88 99.06)
 		)
@@
 	(wire
 		(pts
-			(xy 62.23 29.21) (xy 80.01 29.21)
-		)
-		(stroke
-			(width 0)
-			(type default)
-		)
-	)
-	(wire
-		(pts
 			(xy 41.91 57.15) (xy 41.91 60.96)
 		)
@@
 	(wire
 		(pts
+			(xy 76.2 24.13) (xy 76.2 29.21)
+		)
+		(stroke
+			(width 0)
+			(type default)
+		)
+	)
+	(wire
+		(pts
 			(xy 81.28 85.09) (xy 95.25 85.09)
 		)
@@
 	(wire
 		(pts
+			(xy 67.31 26.67) (xy 67.31 24.13)
+		)
+		(stroke
+			(width 0)
+			(type default)
+		)
+	)
+	(wire
+		(pts
 			(xy 109.22 160.02) (xy 113.03 160.02)
 		)
@@
 	(wire
 		(pts
-			(xy 62.23 26.67) (xy 80.01 26.67)
-		)
-		(stroke
+			(xy 62.23 26.67) (xy 67.31 26.67)
+		)
+		(stroke
+			(width 0)
+			(type default)
+		)
+	)
+	(wire
+		(pts
+			(xy 69.85 26.67) (xy 80.01 26.67)
+		)
+		(stroke

Commit message: dev
Parts:
- removed J1: USB-C input, TerminalBlock_Phoenix:TerminalBlock_Phoenix_MKDS-1,5-2_1x02_P5.00mm_Horizontal, symbol Connector:Screw_Terminal_01x02
- removed J2: Buzzer, TerminalBlock_Phoenix:TerminalBlock_Phoenix_MKDS-1,5-2_1x02_P5.00mm_Horizontal, symbol Connector:Screw_Terminal_01x02
- removed R1: 10k, Resistor_SMD:R_1206_3216Metric_Pad1.30x1.75mm_HandSolder, symbol Device:R
- removed R10, R13, R7: 0R, Resistor_SMD:R_2512_6332Metric_Pad1.40x3.35mm_HandSolder, symbol Device:R
- removed R8: 10k,1206, Resistor_SMD:R_1206_3216Metric_Pad1.30x1.75mm_HandSolder, symbol Device:R
- removed U1: ESP32-C3_SUPERMINI_TH, custom_footprints:MODULE_ESP32-C3_SUPERMINI_TH, symbol Custom_library:ESP32-C3_SUPERMINI_TH
- removed U2: Ai-Thinker-Ra-02, custom_footprints:Ai-Thinker-Ra-01-LoRa BREAKOUT BOARD, symbol RF_Module:Ai-Thinker-Ra-02
- removed U4: (no value), custom_footprints:CKCS BS-01, symbol Custom_library:CKCS_BS-01
- added BT1: Battery, custom_footprints:BHC-CR123A, symbol Device:Battery
- added BZ1: Buzzer, Buzzer_Beeper:Buzzer_12x9.5RM7.6, symbol Device:Buzzer
- added C4: 0805,47uF, Capacitor_SMD:C_0805_2012Metric_Pad1.18x1.45mm_HandSolder, symbol Device:C
- added C5: 0805,47uF (min 10V), Capacitor_SMD:C_0805_2012Metric_Pad1.18x1.45mm_HandSolder, symbol Device:C
- added C6, C7: 47uF, Capacitor_SMD:C_0805_2012Metric_Pad1.18x1.45mm_HandSolder, symbol Device:C
- added C8: 0,1uF, Capacitor_SMD:C_0805_2012Metric_Pad1.18x1.45mm_HandSolder, symbol Device:C
- added C9: 100uF, Capacitor_SMD:C_0805_2012Metric_Pad1.18x1.45mm_HandSolder, symbol Device:C
- added D2: SS14, Diode_SMD:D_SMA, symbol Diode:SS14
- added J1: Conn_01x04_Pin, Connector_PinHeader_2.00mm:PinHeader_1x05_P2.00mm_Vertical, symbol Connector:Conn_01x05_Pin
- added J2: USB-C connector, Connector_JST:JST_PH_B2B-PH-K_1x02_P2.00mm_Vertical, symbol Connector:Conn_01x02_Socket
- added L1: 47uH, CDRH74, Inductor_SMD:L_7.3x7.3_H4.5, symbol Device:L
- added Q2, Q3: AO3401A, Package_TO_SOT_SMD:SOT-23, symbol Transistor_FET:AO3401A
- added R11: 100k,1206, Resistor_SMD:R_1206_3216Metric_Pad1.30x1.75mm_HandSolder, symbol Device:R
- added R12: 10k, Resistor_SMD:R_1206_3216Metric_Pad1.30x1.75mm_HandSolder, symbol Device:R
- added U1: HT7750_C250900, custom_footprints:HT7750, symbol Custom_library:HT7750_C250900
- added U4: E77-900M22S, custom_footprints:COMM-SMD_30P-L20.0-W14.0-P1.27, symbol Custom_library:E77-900M22S
- C2: value 100-220uF -> 100uF; footprint Capacitor_SMD:C_Elec_5x5.4 -> Capacitor_SMD:C_0805_2012Metric_Pad1.18x1.45mm_HandSolder
- R3: value 10k,1206 -> 100k,1206
- R6: value 0R -> 100k,1206; footprint Resistor_SMD:R_2512_6332Metric_Pad1.40x3.35mm_HandSolder -> Resistor_SMD:R_1206_3216Metric_Pad1.30x1.75mm_HandSolder
Connections:
- net +12V is gone; now on net +3.3V: D1.1 (K)
- net +3.3V: now also R2.1, R6.1, BZ1.1 (+), C8.1, C9.1, J1.1 (Pin_1), Q2.3 (D), Q3.2 (S), R12.1, U4.28 (VDD); no longer C2.2, R2.2, U3.2 (VO)
- net +5V: now also C5.1, C7.1, D2.1 (K), J2.2 (Pin_2), Q2.1 (G), R11.2, U1.2 (VOUT)
- net BUZZER: now also Q1.1 (G), R5.1, U4.1 (PB3); no longer R6.2
- net GNDD: now also C2.2, SW1.1, BT1.2 (-), C4.2, C5.2, C6.2, C7.2, C8.2, C9.2, J1.4 (Pin_4), J2.1 (Pin_1), R11.1, U1.1 (GND), U4.15 (GND), U4.27 (GND); no longer C2.1, SW1.2
- net LINK_BUTTON: now also U4.7 (PA0)
- net MODE: now also SW2.2 (B)
- net SENSOR: now also J3.2 (Pin_2), R2.2, U4.8 (PA1)
- net at R9.2: now also Q1.3 (D); no longer R6.1
- net at R4.2: now also SW1.2; no longer SW1.1
- net at D1.2 (A): now also U3.2 (VO), C6.1; no longer Q1.3 (D)
- new net: BZ1.2 (-), R12.2, R9.1
- new net: C4.1, L1.1, Q3.3 (D)
- new net: D2.2 (A), L1.2, U1.3 (LX)
- new net: BT1.1 (+), Q2.2 (S)
- new net HT7750_EN: Q3.1 (G), R6.2, U4.23 (PB2)
- new net NRST: C2.1, J1.5 (Pin_5), U4.17 (NRST)
- new net SWCLK: J1.3 (Pin_3), U4.30 (SWCLK)
- new net SWDIO: J1.2 (Pin_2), U4.29 (SWDIO)
- new net UART_TX: U4.9 (PA2)
- no-connect marks 10 -> 19
Other:
- moved on the sheet: C1, J3, Q1, R2, R3, R4, R5, SW1, SW2, U3
